File: ADSR_Envelope_THT/ADSR_Envelope_THT.kicad_pcb (KiCad board)
At the start: 2 copper layers, 51 parts, among them J1 AudioJack1_Switch, J2 AudioJack1_Switch, J3 Conn_02x08_Odd_Even, J4 AudioJack1_Switch, Q1 2N7000, Q2 2N3904, Q3 2N3904, Q4 2N3904, SW1 SW_Push, SW2 SW_DPDT_x2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

Commit message: ADSR Envelope
Updated the Schematic for the ADSR Envilope and started on the PCB layout
Parts:
- added J5: Conn_01x12, Pin_Headers:Pin_Header_Straight_1x12_Pitch2.54mm, F.Cu at (42.0, 73.0)
- added J6: Conn_01x12, Pin_Headers:Pin_Header_Straight_1x12_Pitch2.54mm, F.Cu at (38.0, 37.0)
- added J7: Conn_01x12, Pin_Headers:Pin_Header_Straight_1x12_Pitch2.54mm, F.Cu at (18.0, 37.0)
- added J8: Conn_01x12, Pin_Headers:Pin_Header_Straight_1x12_Pitch2.54mm, F.Cu at (22.0, 37.0)
- SW1: footprint SamacSys_Parts:FSMRACDAH -> Custom_Library:SW_Tactile_TE_FSMRACDAH
- moved C1 463.7 mm to (-246.7, 3.28)
- moved C2 463.7 mm to (-246.7, 7.53)
- moved C3 463.7 mm to (-255.4, 27.9)
- moved C4 463.7 mm to (-266.1, 34.2)
- moved C5 463.7 mm to (-268.5, 49.5)
- moved C6 463.7 mm to (-254.2, 34.0)
- moved C7 463.7 mm to (-263.3, 40.4)
- moved C8 463.7 mm to (-246.1, 24.6)
- moved D4 463.7 mm to (-275.3, 44.2)
- moved J3 463.7 mm to (-340.6, 3.48)
- moved Q1 463.7 mm to (-246.7, 12.9)
- moved Q3 463.7 mm to (-277.9, 51.0)
- moved Q4 463.7 mm to (-248.3, 18.7)
- moved R10 463.7 mm to (-260.0, 3.28)
- moved R12 463.7 mm to (-260.0, 7.53)
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Connections:
- C3 pad 1: Net-(C3-Pad1) -> Speed3
- C4 pad 1: Net-(C4-Pad1) -> Speed2
- D2 pad 1: Net-(D2-Pad1) -> RELout
- D3 pad 1: Net-(D3-Pad1) -> Button
- D4 pad 2: Net-(D4-Pad2) -> RELin
- D5 pad 1: Net-(D5-Pad1) -> LEDin
- D5 pad 2: Net-(D5-Pad2) -> LEDout
- D6 pad 1: Net-(D5-Pad2) -> Net-(D6-Pad1)
- D6 pad 2: Net-(D5-Pad1) -> Net-(D6-Pad2)
- J1 pad 1: GND -> /GND_In
- J1 pad 2: Gate -> Net-(J1-Pad2)
- J2 pad 1: GND -> /GND_Out
- J3 pad 13: Gate -> GateIn
- J3 pad 14: Gate -> GateIn
- J4 pad 1: GND -> /GND_Out
- Q1 pad 3: Net-(Q1-Pad3) -> SUSin
- Q3 pad 2: Net-(D3-Pad1) -> Button
- R1 pad 1: +12v -> /12VDC_In
- R10 pad 1: Net-(R10-Pad1) -> Speed1
- R12 pad 1: Net-(D3-Pad1) -> Button
- R12 pad 2: Net-(J1-Pad3) -> GateOut
- R13 pad 1: Net-(D2-Pad1) -> Net-(J7-Pad12)
- R14 pad 1: Net-(J1-Pad3) -> GateOut
- R16 pad 1: Net-(J2-Pad3) -> Net-(J5-Pad8)
- R16 pad 2: THR -> Net-(J2-Pad3)
- R17 pad 1: THR -> ADSRout
- R18 pad 1: Net-(J4-Pad3) -> Net-(J5-Pad9)
- R18 pad 2: Net-(R18-Pad2) -> Net-(J4-Pad3)
- R19 pad 1: Net-(R18-Pad2) -> ADSRInvert
- R21 pad 1: Net-(D5-Pad1) -> LEDin
- R21 pad 2: THR -> ADSRout
- R4 pad 1: +12v -> /12VDC_Out
- R5 pad 1: Net-(D2-Pad1) -> RELout
- R5 pad 2: Net-(R5-Pad2) -> DECout
- R8 pad 2: Net-(R8-Pad2) -> ATTout
- R9 pad 1: Net-(D3-Pad1) -> Net-(J5-Pad2)
- RV1 pad 2: Net-(RV1-Pad2) -> Net-(J7-Pad9)
- RV1 pad 3: Net-(Q1-Pad3) -> Net-(J7-Pad10)
- RV2 pad 2: Net-(R5-Pad2) -> Net-(J7-Pad7)
- RV3 pad 1: Net-(RV3-Pad1) -> Net-(J7-Pad4)
- RV3 pad 2: Net-(R8-Pad2) -> Net-(J7-Pad5)
- RV4 pad 1: Net-(D4-Pad2) -> Net-(J7-Pad11)
- SW1 pad 1: Net-(R9-Pad2) -> Net-(R4-Pad2)
- SW1 pad 2: Net-(R4-Pad2) -> Net-(R9-Pad2)
- SW2 pad 1: Net-(R8-Pad2) -> Net-(J5-Pad3)
- SW2 pad 2: Net-(R10-Pad1) -> Net-(J5-Pad4)
- SW2 pad 4: Net-(C4-Pad1) -> Net-(J5-Pad7)
- SW2 pad 5: Net-(D2-Pad1) -> Net-(J5-Pad6)
- SW2 pad 6: Net-(C3-Pad1) -> Net-(J5-Pad5)
- U1 pad 1: THR -> ADSRout
- U1 pad 12: Net-(RV1-Pad2) -> SUSout
- U1 pad 13: Net-(D1-Pad1) -> DECin
- U1 pad 14: Net-(D1-Pad1) -> DECin
- U1 pad 2: THR -> ADSRout
- U1 pad 3: Net-(D2-Pad1) -> RELout
- U1 pad 6: Net-(D5-Pad1) -> LEDin
- U1 pad 7: Net-(D5-Pad2) -> LEDout
- U1 pad 8: Net-(R18-Pad2) -> ADSRInvert
- U2 pad 3: Net-(RV3-Pad1) -> ATTin
- U2 pad 6: THR -> ADSRout
Routing:
- net Net-(J1-Pad3): track 0.00 -> 36.4 mm
- net Net-(J7-Pad11): track 0.00 -> 34.6 mm
- net Net-(J5-Pad3): track 0.00 -> 28.9 mm
- net Net-(J1-Pad2): track 0.00 -> 28.1 mm
- net Net-(J7-Pad9): track 0.00 -> 27.8 mm
- net Net-(J5-Pad4): track 0.00 -> 27.2 mm
- net Net-(J5-Pad2): track 0.00 -> 27.1 mm
- net Net-(J7-Pad10): track 0.00 -> 26.5 mm
- net Net-(J7-Pad5): track 0.00 -> 22.8 mm
- net Net-(J7-Pad4): track 0.00 -> 22.4 mm
- net /12VDC_Out: track 0.00 -> 21.4 mm
- net Net-(J5-Pad6): track 0.00 -> 21.1 mm
- net Net-(J5-Pad5): track 0.00 -> 20.3 mm
- net Net-(J5-Pad7): track 0.00 -> 20.3 mm
- net Net-(J7-Pad12): track 0.00 -> 20.0 mm
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- added copper zone on B.Cu, net /GND_In
- added copper zone on F.Cu, net /GND_In
Other:
- board outline added: 60 x 110 mm
- net class PWR added: clearance 0.2, trace_width 0.5, via_dia 0.8, via_drill 0.4

Commit message: ADSR Envelope
Finished the PCB design on the ADSR Envelope
Parts:
- moved R5 388.9 mm to (48.0, 92.0)
- moved J3 372.7 mm to (22.0, 90.0)
- moved R2 362.9 mm to (52.0, 4.00), turned to 180 degrees
- moved U1 358.2 mm to (36.0, 67.0)
- moved R17 349.6 mm to (58.3, 77.0), turned to 180 degrees
- moved R15 348.9 mm to (46.0, 30.0), turned to 180 degrees
- moved R19 344.2 mm to (48.0, 97.0)
- moved R20 342.0 mm to (48.0, 87.0)
- moved R8 341.9 mm to (48.0, 82.0)
- moved R11 334.9 mm to (48.0, 107.0)
- moved R3 334.4 mm to (32.0, 58.0), turned to 90 degrees
- moved R6 331.6 mm to (27.0, 4.00)
- moved D2 330.4 mm to (52.5, 60.0), turned to 180 degrees
- moved R21 325.3 mm to (32.0, 72.0), turned to 90 degrees
- moved R10 323.5 mm to (48.0, 102.0)
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Connections:
- J5 pad 10: /GND_Out -> Net-(J5-Pad10)
- J5 pad 11: Net-(D6-Pad1) -> Net-(J5-Pad11)
- J5 pad 12: Net-(D6-Pad2) -> /GND_Out
- J5 pad 8: Net-(J5-Pad8) -> Net-(D6-Pad1)
- J5 pad 9: Net-(J5-Pad9) -> Net-(D6-Pad2)
- J6 pad 10: GND -> ADSRout
- J6 pad 11: LEDout -> ADSRInvert
- J6 pad 12: LEDin -> GND
- J6 pad 8: ADSRout -> LEDout
- J6 pad 9: ADSRInvert -> LEDin
- R16 pad 1: Net-(J5-Pad8) -> Net-(J5-Pad10)
- R18 pad 1: Net-(J5-Pad9) -> Net-(J5-Pad11)
Routing:
- net +12v: track 0.00 -> 153.3 mm
- net GateIn: track 0.00 -> 118.3 mm, vias 0 -> 2
- net Net-(C1-Pad2): track 0.00 -> 99.4 mm
- net ATTout: track 0.00 -> 89.6 mm, vias 0 -> 2
- net RELout: track 0.00 -> 88.4 mm
- net Net-(C1-Pad1): track 0.00 -> 80.6 mm
- net Speed1: track 0.00 -> 69.2 mm
- net -12v: track 0.00 -> 69.0 mm
- net Speed3: track 0.00 -> 67.6 mm
- net ADSRout: track 0.00 -> 65.7 mm
- net GateOut: track 0.00 -> 49.2 mm
- net ADSRInvert: track 0.00 -> 48.6 mm
- net Net-(D2-Pad2): track 0.00 -> 48.6 mm
- net SUSin: track 0.00 -> 45.5 mm
- net DECout: track 0.00 -> 41.6 mm
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- added copper zone on B.Cu, net /GND_Out
- added copper zone on F.Cu, net /GND_Out
- added copper zone on B.Cu, net GND
- added copper zone on F.Cu, net GND
Other:
- board size 60 x 110 mm -> 80 x 110 mm
