File: Through Hole Designs/ADSR_Envelope_THT/ADSR_Envelope_THT.sch (KiCad schematic (older format))
At the start: 55 parts, among them J1 AudioJack1_Switch, J2 AudioJack1_Switch, J3 Conn_02x08_Odd_Even, J4 AudioJack1_Switch, J5 Conn_01x12, J6 Conn_01x12, J7 Conn_01x12, J8 Conn_01x12, Q1 2N7000, Q2 2N3904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

Commit message: KiCAD Update Test
Updated KiCad and tested loading a file
Parts:
- removed U2: ICM7555, Housings_DIP:DIP-8_W7.62mm_Socket, symbol Timer:ICM7555
- added U2: ICM7555xB, Housings_DIP:DIP-8_W7.62mm_Socket, symbol Timer:ICM7555xB
Connections:
- net +12v: now also U2.8 (VCC)
- net ADSRout: now also U2.6 (THR)
- net ATTin: now also U2.3 (Q)
- net GND: now also U2.1 (GND)
- net at C1.1, D4.1 (K), Q4.3 (C)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: now also U2.4 (R)
- net at Q2.3 (C), R3.2: now also U2.2 (TR)
- net at C2.2: now also U2.5 (CV)
- net at Q1.1 (S): now also U2.7 (DIS)
Changed lines of the file:
@@
 	4450 2650 4400 2650
 Connection ~ 4450 2500
-$Comp
-L Timer:ICM7555 U2
-U 1 1 5F3A309B
-P 6100 2050
-F 0 "U2" H 6100 2631 50  0000 C CNN
-F 1 "ICM7555" H 6100 2540 50  0000 C CNN
-F 2 "Housings_DIP:DIP-8_W7.62mm_Socket" H 6100 2050 50  0001 C CNN
-F 3 "http://www.intersil.com/content/dam/Intersil/documents/icm7/icm7555-56.pdf" H 6100 2050 50  0001 C CNN
-	1    6100 2050
-	1    0    0    -1
-$EndComp
 Wire Wire Line
 	5600 1850 5300 1850
@@
 Wire Wire Line
 	5800 6000 5800 7500
+$Comp
+L Timer:ICM7555xB U2
+U 1 1 5FD4D518
+P 6100 2050
+F 0 "U2" H 6100 2631 50  0000 C CNN
+F 1 "ICM7555xB" H 6100 2540 50  0000 C CNN
+F 2 "Housings_DIP:DIP-8_W7.62mm_Socket" H 6950 1650 50  0001 C CNN
+F 3 "http://www.intersil.com/content/dam/Intersil/documents/icm7/icm7555-56.pdf" H 6950 1650 50  0001 C CNN
+	1    6100 2050
+	1    0    0    -1
+$EndComp
 $EndSCHEMATC
