File: Through Hole Designs/ADSR_Envelope_THT/ADSR_Envelope_THT.kicad_pcb (KiCad board)
At the start: 2 copper layers, 80 x 110 mm, 55 parts, among them J1 AudioJack1_Switch, J2 AudioJack1_Switch, J3 Conn_02x08_Odd_Even, J4 AudioJack1_Switch, J5 Conn_01x12, J6 Conn_01x12, J7 Conn_01x12, J8 Conn_01x12, Q1 2N7000, Q2 2N3904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

Commit message: KiCAD 6.0 Update
Updated all the project files to Version 6.0 of KiCAD.  No change to Gerbers or Schematics.
Other:
- net class Default removed
- net class PWR removed
