File: Through Hole Designs/LFO_THT/LFO_THT.kicad_pcb (KiCad board)
At the start: 2 copper layers, 100 x 110 mm, 79 parts, among them J1 AudioJack1_Switch, J10 AudioJack1_Switch, J11 AudioJack1_Switch, J2 Conn_01x12, J3 Conn_01x12, J4 AudioJack1_Switch, J5 AudioJack1_Switch, J6 AudioJack1_Switch, J7 Conn_02x08_Odd_Even, J8 Conn_01x07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

Commit message: KiCAD 6.0 Update
Updated all the project files to Version 6.0 of KiCAD.  No change to Gerbers or Schematics.
Other:
- net class Default removed
- net class PWR removed
