File: Surface Mount Designes/LFO/LFO.sch (KiCad schematic (older format))
At the start: 79 parts, among them J1 AudioJack1_Switch, J10 AudioJack1_Switch, J11 AudioJack1_Switch, J2 Conn_01x12, J3 Conn_01x12, J4 AudioJack1_Switch, J5 AudioJack1_Switch, J6 AudioJack1_Switch, J7 Conn_02x08_Odd_Even, J8 Conn_01x07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

Commit message: Comb
Finished The Schematic for the Comb Filter and started on the Surface Mount PCB design
Parts:
- U1: symbol Timer:ICM7555 -> LFO-rescue:ICM7555-Timer
Changed lines of the file:
@@
 $EndComp
 $Comp
-L Timer:ICM7555 U1
+L LFO-rescue:ICM7555-Timer U1
 U 1 1 5FFAE60D
 P 5650 1400
