File: Unfinished Designs/Comb_Filter/Comb_Filter.sch (KiCad schematic (older format))
At the start: 164 parts, among them J2 Conn_02x05_Odd_Even, U1 TL074, U2 TL074, U3 TL074, U4 TL074

Commit message: Comb
Finished The Schematic for the Comb Filter and started on the Surface Mount PCB design
Parts:
- C1, C10, C12, C14, C16, C17, C19, C2, C21, C27, C28, C29, C3, C32, C35, C36, C37, C4, C6, C7: renamed from C?; footprint (none) -> Capacitors_SMD:C_1210_HandSoldering
- C11, C15, C18, C22: renamed from C?; value 22uF -> 0.0047uF; footprint (none) -> Capacitors_SMD:C_1210_HandSoldering
- C13, C8: renamed from C?; value 22uF -> 820pF; footprint (none) -> Capacitors_SMD:C_1210_HandSoldering
- C20, C26: renamed from C?; value 22uF -> 470pF; footprint (none) -> Capacitors_SMD:C_1210_HandSoldering
- C23, C30: renamed from C?; value 22uF -> 0.022uF; footprint (none) -> Capacitors_SMD:C_1210_HandSoldering
- C24, C25, C31: renamed from C?; value 22uF -> 0.0022uF; footprint (none) -> Capacitors_SMD:C_1210_HandSoldering
- C33, C38, C5, C9: renamed from C?; value 22uF -> 0.01uF; footprint (none) -> Capacitors_SMD:C_1210_HandSoldering
- C34: renamed from C?; value 22uF -> 0.0015uF; footprint (none) -> Capacitors_SMD:C_1210_HandSoldering
- C39, C44: renamed from C?; footprint (none) -> Capacitors_SMD:CP_Elec_5x5.8
- C40, C41, C42, C43: renamed from C?; footprint (none) -> Capacitors_SMD:CP_Elec_6.3x5.8
- J1, J10, J11, J12, J13, J3, J4, J5, J6, J7, J8, J9: renamed from J?; footprint (none) -> Custom_Library:Mono_Jack_3.5mm_Switch_Switchcraft_35RAPC2AH3
- J2: footprint (none) -> Pin_Headers:Pin_Header_Straight_2x05_Pitch2.54mm
- R1, R10, R11, R14, R15, R16, R17, R18, R19, R2, R22, R23, R24, R25, R26, R29, R3, R30, R31, R33, R34, R36, R37, R38, R39, R4, R40, R41, R42, R44, R45, R47, R49, R5, R50, R53, R54, R59, R6, R64, R66, R67, R68, R69, R7, R72, R75, R76, R77, R8, R9: renamed from R?; footprint (none) -> Resistors_SMD:R_1210_HandSoldering
- R12, R27, R43, R55, R56, R70: renamed from R?; value 56k -> 15k; footprint (none) -> Resistors_SMD:R_1210_HandSoldering
- R13, R28, R46, R57, R58, R71: renamed from R?; value 56k -> 220; footprint (none) -> Resistors_SMD:R_1210_HandSoldering
- R20, R32, R48, R62, R73: renamed from R?; value 56k -> 150k; footprint (none) -> Resistors_SMD:R_1210_HandSoldering
- R21, R35, R51, R74: renamed from R?; value 56k -> 180k; footprint (none) -> Resistors_SMD:R_1210_HandSoldering
- R52: renamed from R?; value 65k -> 64k9; footprint (none) -> Resistors_SMD:R_1210_HandSoldering
- R60: renamed from R?; value 56k -> 91k; footprint (none) -> Resistors_SMD:R_1210_HandSoldering
- R61: renamed from R?; value 56k -> 68k; footprint (none) -> Resistors_SMD:R_1210_HandSoldering
- R63: renamed from R?; value 56k -> 100k; footprint (none) -> Resistors_SMD:R_1210_HandSoldering
- R65: renamed from R?; value 4.7k -> 4k7; footprint (none) -> Resistors_SMD:R_1210_HandSoldering
- RV1, RV11, RV12, RV15, RV3, RV8: renamed from RV?; value R_POT -> 100k; footprint (none) -> Custom_Library:PVG5A
- RV10, RV13, RV14, RV16, RV2, RV5: renamed from RV?; value R_POT -> 20k; footprint (none) -> Custom_Library:PVG5A
- RV4, RV6, RV7, RV9: renamed from RV?; footprint (none) -> Custom_Library:PVG5A
- U1, U2, U3, U4: footprint (none) -> Housings_SOIC:SOIC-14_3.9x8.7mm_Pitch1.27mm
Connections:
- net 1k: now also R13.2
- net 1k4: now also R28.2
- net 2k: now also R46.2
- net 3k5: now also R58.2
- net 500: now also R57.2
- net 700: now also R71.2
- net GND: now also R21.1, R35.1, R51.1, R62.1, R63.1, R74.1
- net at C3.1, C35.2, R4.1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: now also C15.2, C22.2, C31.2, C9.2, R12.2, R27.2, R43.2, R56.2
- net at U1.12 (+): now also R21.2
- net at U1.13 (-): now also C8.1, RV1.3
- net at U1.14: now also C5.1, R13.1, RV2.3
- net at U3.10 (+): now also R63.2
- net at U3.8: now also C24.1, R58.1, RV14.3
- net at U3.9 (-): now also C26.1, RV12.3
- net at U3.1: now also C11.1, R28.1, RV5.3
- net at U3.2 (-): now also C13.1, RV3.3
- net at U3.3 (+): now also R35.2
- net at U3.5 (+): now also R51.2
- net at U3.6 (-): now also C20.1, RV8.3
- net at U3.7: now also C18.1, R46.1, RV10.3
- net at U2.10 (+): now also R62.2
- net at U2.8: now also C23.1, R57.1, RV13.3
- net at U2.9 (-): now also C25.1, RV11.3
- net at U2.12 (+): now also R74.2
- net at U2.13 (-): now also C34.1, RV15.3
- net at U2.14: now also C33.1, R71.1, RV16.3
- net at C16.2, C2.1, C21.2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: now also C30.2, C38.2, R55.2, R70.2
- net at C23.2: now also C25.2, R55.1
- net at C30.1: now also R60.2, RV13.1, RV13.2
- net at R60.1: now also RV11.2
- net at C24.2: now also C26.2, R56.1
- net at C31.1: now also R61.2, RV14.1, RV14.2
- net at R61.1: now also RV12.2
- net at C33.2: now also C34.2, R70.1
- net at C38.1: now also R73.2, RV16.1, RV16.2
- net at R73.1: now also RV15.2
- net at C5.2: now also C8.2, R12.1
- net at C9.1: now also R20.2, RV2.1, RV2.2
- net at R20.1: now also RV1.2
- net at C11.2: now also C13.2, R27.1
- net at C15.1: now also R32.2, RV5.1, RV5.2
- net at R32.1: now also RV3.2
- net at C18.2: now also C20.2, R43.1
- net at C22.1: now also R48.2, RV10.1, RV10.2
- net at R48.1: now also RV8.2
Other:
- note added: "1 kHz"
- note added: "1.4 kHz"
- note added: "2 kHz"
- note added: "3.5 kHz"
- note added: "500 Hz"
- note added: "700 Hz"
- note added: "Greater Then 7 kHz"
- moved on the sheet: R13, R21, R28, R35, R46, R51, R57, R58, R62, R63, R71, R74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

Commit message: 1-29-2021 Comb
Started Layout of Comb Filter
Parts:
- added J14, J15, J16, J17: Conn_01x07, Pin_Headers:Pin_Header_Straight_1x07_Pitch2.54mm, symbol Connector_Generic:Conn_01x07
Connections:
- net 1k: no longer J8.3
- net 1k4: no longer J9.3
- net 200: no longer J4.3
- net 2k: no longer J10.3
- net 350: no longer J5.3
- net 3k5: no longer J11.3
- net 500: no longer J6.3
- net 700: no longer J7.3
- net <100: no longer J3.3
- net >7k: no longer J12.3
- net GND: now also J14.7 (Pin_7), J16.7 (Pin_7); no longer J1.1, J1.2, J10.1, J11.1, J12.1, J13.1, J3.1, J4.1, J5.1, J6.1, J7.1, J8.1, J9.1
- net at J13.3: now also J17.6 (Pin_6); no longer R64.1
- net <100_Out: now reaches FADE1.2, R7.1
- net <100_Out: now also J14.1 (Pin_1)
- net 200_Out: now reaches FADE2.2, R9.1
- net 200_Out: now also J16.1 (Pin_1)
- net 350_Out: now reaches FADE3.2, R15.1
- net 350_Out: now also J14.2 (Pin_2)
- net 500_Out: now reaches FADE4.2, R23.1
- net 500_Out: now also J16.2 (Pin_2)
- net 700_Out: now reaches FADE5.2, R25.1
- net 700_Out: now also J14.3 (Pin_3)
- net 1k_Out: now reaches FADE6.2, R30.1
- net 1k_Out: now also J16.3 (Pin_3)
- net 1k4_Out: now reaches FADE7.2, R36.1
- net 1k4_Out: now also J14.4 (Pin_4)
- net 2k_Out: now reaches FADE8.2, R39.1
- net 2k_Out: now also J16.4 (Pin_4)
- net 3k5_Out: now reaches FADE9.2, R41.1
- net 3k5_Out: now also J14.5 (Pin_5)
- net >7k_Out: now reaches FADE10.2, R49.1
- net >7k_Out: now also J16.5 (Pin_5)
- net at J1.3: now also J15.6 (Pin_6); no longer C1.2
- new net: J10.1, J12.1, J13.1, J17.7 (Pin_7), J4.1, J6.1, J8.1
- new net: J15.1 (Pin_1), J3.3
- new net: J15.2 (Pin_2), J5.3
- new net: J15.3 (Pin_3), J7.3
- new net: J15.4 (Pin_4), J9.3
- new net: J11.3, J15.5 (Pin_5)
- new net: J1.1, J1.2, J11.1, J15.7 (Pin_7), J3.1, J5.1, J7.1, J9.1
- new net: J17.1 (Pin_1), J4.3
- new net: J17.2 (Pin_2), J6.3
- new net: J17.3 (Pin_3), J8.3
- new net: J10.3, J17.4 (Pin_4)
- new net: J12.3, J17.5 (Pin_5)
- new net Input: C1.2, J14.6 (Pin_6)
- new net Output: J16.6 (Pin_6), R64.1
Other:
- note added: "Faders"
- note added: "Left Side Riser"
- note added: "Right Side Riser"
- note removed: "Faders and Individual Outputs"
- note removed: "Input"
- moved on the sheet: C27, C28, C29, FADE10A, FADE10B, FADE1A, FADE1B, FADE2A, FADE2B, FADE3A, FADE3B, FADE4A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
