File: Surface Mount Designes/Patch_Bay/Patch_Bay.kicad_pcb (KiCad board)
At the start: 2 copper layers, 25 x 100 mm, 9 parts, among them J1 AudioJack1_Switch, J2 AudioJack1_Switch, J3 AudioJack1_Switch, J4 AudioJack1_Switch, J5 AudioJack1_Switch, J6 AudioJack1_Switch, J7 AudioJack1_Switch, J8 AudioJack1_Switch, J9 Conn_02x06_Odd_Even

Commit message: KiCAD 6.0 Update
Updated all the project files to Version 6.0 of KiCAD.  No change to Gerbers or Schematics.
Other:
- net class Default removed
