File: Surface Mount Designes/VCF/VCF.kicad_pcb (KiCad board)
At the start: 2 copper layers, 54 x 100 mm, 48 parts, among them J1 AudioJack1_Switch, J2 AudioJack1_Switch, J3 Conn_01x04, J4 Conn_01x04, J5 Conn_02x08_Odd_Even, J6 AudioJack1_Switch, Q1 BC818, Q2 BC818, Q3 BC818, Q4 BC818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

Commit message: KiCAD 6.0 Update
Updated all the project files to Version 6.0 of KiCAD.  No change to Gerbers or Schematics.
Other:
- net class Default removed
- net class PWR removed
