File: Through Hole Designs/Logic_Gates_THT/NAND_THT/NAND_THT.kicad_pcb (KiCad board)
At the start: 2 copper layers, 100 x 100 mm, 89 parts, among them J1 AudioJack1_Switch, J10 Conn_01x08, J11 Conn_01x08, J12 Conn_01x08, J13 Conn_02x08_Odd_Even, J14 Conn_01x12, J15 Conn_01x12, J16 AudioJack1_Switch, J17 AudioJack1_Switch, J18 AudioJack1_Switch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

Commit message: KiCAD 6.0 Update
Updated all the project files to Version 6.0 of KiCAD.  No change to Gerbers or Schematics.
Other:
- net class Default removed
- net class PWR removed
