File: Through Hole Designs/Noise_Gen_THT/Noise_Gen_THT.kicad_pcb (KiCad board)
At the start: 2 copper layers, 30 x 100 mm, 24 parts, among them J1 AudioJack1_Switch, J2 AudioJack1_Switch, J5 Conn_02x05_Odd_Even, Q1 2N3904, U1 TL072

Commit message: KiCAD 6.0 Update
Updated all the project files to Version 6.0 of KiCAD.  No change to Gerbers or Schematics.
Other:
- net class Default removed
- net class PWR removed
