File: Through Hole Designs/Notch_Filter_THT/Notch_Filter_THT.kicad_pcb (KiCad board)
At the start: 2 copper layers, 30 x 100 mm, 29 parts, among them J1 AudioJack1_Switch, J2 AudioJack1_Switch, J3 Conn_02x08_Odd_Even, J4 AudioJack1_Switch, Q1 2N3904, Q2 2N3904, Q3 2N3904, Q4 2N3904, U1 TL074

Commit message: KiCAD 6.0 Update
Updated all the project files to Version 6.0 of KiCAD.  No change to Gerbers or Schematics.
Other:
- net class Default removed
- net class PWR removed
