File: Through Hole Designs/Power_Distribution_THT/Power_Distribution_THT.kicad_pcb (KiCad board)
At the start: 2 copper layers, 210 x 80 mm, 37 parts, among them J1 Conn_02x08_Odd_Even, J10 Conn_02x08_Odd_Even, J11 Conn_02x05_Odd_Even, J12 Conn_02x05_Odd_Even, J13 Conn_02x05_Odd_Even, J14 Conn_02x05_Odd_Even, J15 Conn_02x05_Odd_Even, J16 Conn_02x05_Odd_Even, J17 Conn_02x05_Odd_Even, J18 Conn_02x05_Odd_Even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

Commit message: KiCAD 6.0 Update
Updated all the project files to Version 6.0 of KiCAD.  No change to Gerbers or Schematics.
Other:
- net class Default removed
- net class PWR removed
