File: Through Hole Designs/Power_Supply_THT/Power_Supply_THT.kicad_pcb (KiCad board)
At the start: 2 copper layers, 200 x 120 mm, 57 parts, among them J1 Hot_In, J2 Netral_IN, J3 Nutral_Out, J4 Hot_Out, J5 18VAC_1, J6 CT, J7 18VAC_2, J8 Screw_Terminal_01x04, U1 L7812, U2 L7812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

Commit message: KiCAD 6.0 Update
Updated all the project files to Version 6.0 of KiCAD.  No change to Gerbers or Schematics.
Other:
- net class Default removed
- net class HighVolt removed
- net class PWR removed
- net class PreReg removed
