File: Through Hole Designs/Power_Supply_THT/Power_Supply_THT.kicad_sch (KiCad schematic)
At the start: 49 parts, among them J1 Hot_In, J2 Netral_IN, J3 Nutral_Out, J4 Hot_Out, J5 18VAC_1, J6 CT, J7 18VAC_2, J8 Screw_Terminal_01x04, U1 L7812, U2 L7812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

Commit message: KiCad 9.0 Update
Installed KiCad 9.0 and updated all the files to latest version before continuing work on the designs.
Parts:
- C8: value 0.1uF -> 0.1uF
